File: hardware/microNES_pcb_v0.1/microNES_pcb_v0.1.kicad_pcb (KiCad board)
At the start: 4 copper layers, 72.3 x 70 mm, 105 parts, among them J1 USB_C_Receptacle_USB2.0_16P, J3 HDMI_E, J4 SM03B-SRSS-TB, J5 Conn_01x05, Q1 2N7002, SW3 PTS810SJM250SMTRLFS, SW4 PTS810SJM250SMTRLFS, U1 RP2350_60QFN, U2 AMS1117-3.3, U3 W25Q128JVS, U5 AMS1117-3.3, Y1 ABM8-272-T3

Commit message: make more games work and also update hardware pcb to .v2
Parts:
- removed G***: LOGO, microNES_footprints:logo-silkscreen
- removed J5: Conn_01x05, microNES_footprints:CONN-SMD_S5B-PH-SM4-TB-LF-SN
- added H2: MountingHole, MountingHole:MountingHole_2.7mm_M2.5, F.Cu at (64.4, 94.1)
- added REF**: logo2-silkscreen, microNES_footprints:logo2-silkscreen, F.Cu at (81.9, 131.6)
- added TP10: ~, TestPoint:TestPoint_Pad_1.5x1.5mm, F.Cu at (122.0, 112.6)
- added TP11: ~, TestPoint:TestPoint_Pad_1.5x1.5mm, F.Cu at (131.2, 112.6)
- added TP8: ~, TestPoint:TestPoint_Pad_1.5x1.5mm, F.Cu at (114.0, 113.0)
- added TP9: ~, TestPoint:TestPoint_Pad_1.5x1.5mm, F.Cu at (116.8, 112.4)
- moved H3 49.3 mm to (64.2, 117.6)
- moved R40 34.8 mm to (66.1, 72.1)
- moved U8 29.7 mm to (63.8, 69.7)
- moved R10 24.8 mm to (92.0, 82.9), turned to 90 degrees
- moved J3 24.6 mm to (99.0, 72.6), turned to 90 degrees
- moved TP7 24.3 mm to (70.2, 75.0)
- moved R26 22.6 mm to (93.6, 82.9), turned to 90 degrees
- moved R27 20.4 mm to (95.2, 82.9), turned to 90 degrees
- moved TP3 18.3 mm to (73.4, 75.0)
- moved R28 18.3 mm to (96.8, 82.9), turned to 90 degrees
- moved R29 16.2 mm to (98.3, 82.9), turned to 90 degrees
- moved H1 15.7 mm to (157.0, 69.9)
- moved R30 14.1 mm to (99.9, 82.9), turned to 90 degrees
- moved H4 12.8 mm to (157.3, 132.2)
- moved R31 12.1 mm to (101.5, 82.9), turned to 90 degrees
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Connections:
- AV1 pad 1: /ADAC_OUT -> GND
- AV1 pad 2: GND -> /ADAC_OUT
- AV2 pad 1: /VDAC_OUT -> GND
- AV2 pad 2: GND -> /VDAC_OUT
- R40 pad 1: Net-(U8-RST_OUT) -> Net-(U8-LED_K)
- R40 pad 2: /RST_BTN -> /PWR_LED
- U8 pad 4: Net-(U8-RST_OUT) -> /RST_BTN
- U8 pad 5: /PWR_LED -> Net-(U8-LED_K)
Routing:
- net /NES_DATA_1: track 71.6 -> 26.8 mm, vias 4 -> 2
- net /RST_BTN: track 38.3 -> 73.7 mm, vias 3 -> 2
- net /NES_CLOCK: track 84.0 -> 51.7 mm
- net VBUS: track 69.6 -> 39.1 mm, vias 8 -> 7
- net /PWR_LED: track 48.8 -> 77.4 mm, vias 3 -> 2
- net /NES_LATCH: track 77.6 -> 50.1 mm
- net /GPIO18: track 32.4 -> 58.7 mm
- net /GPIO19: track 32.6 -> 58.7 mm
- net /GPIO16: track 31.9 -> 52.6 mm
- net /GPIO17: track 32.2 -> 52.2 mm
- net /GPIO14: track 17.2 -> 33.1 mm
- net /GPIO15: track 17.4 -> 33.2 mm
- net /GPIO12: track 16.7 -> 28.1 mm
- net /VDAC_OUT: track 40.8 -> 29.5 mm
- net /GPIO13: track 17.1 -> 28.1 mm
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- added copper zone on In2.Cu, net /VBUS_RAW
Other:
- board size 72.3 x 70 mm -> 101.6 x 70 mm
