File: hardware/microNES_pcb_v0.1/microNES_pcb_v0.1.kicad_sch (KiCad schematic)
At the start: 106 parts, among them J1 USB_C_Receptacle_USB2.0_16P, J3 HDMI_E, J4 SM03B-SRSS-TB, J5 Conn_01x05, Q1 2N7002, SW3 PTS810SJM250SMTRLFS, SW4 PTS810SJM250SMTRLFS, U1 RP2350_60QFN, U2 AMS1117-3.3, U3 W25Q128JVS, U5 AMS1117-3.3, Y1 ABM8-272-T3

Commit message: make more games work and also update hardware pcb to .v2
Parts:
- removed J5: Conn_01x05, microNES_footprints:CONN-SMD_S5B-PH-SM4-TB-LF-SN, symbol microNES_symbols:S5B-PH-SM4-TB
- added H2: MountingHole, MountingHole:MountingHole_2.7mm_M2.5, symbol Mechanical:MountingHole
- added TP10, TP11, TP8, TP9: (no value), TestPoint:TestPoint_Pad_1.5x1.5mm, symbol Connector:TestPoint
- Card1: LCSC (none) -> C393941; LCSC Part C393941 -> (none)
- R24: LCSC C2784782 -> C25076
Connections:
- net ADAC_OUT: now also AV1.2; no longer AV1.1
- net GND: now also AV1.1, AV2.1; no longer AV1.2, AV2.2
- net NES_CLOCK: now also TP8.1
- net NES_DATA_1: now also TP10.1
- net NES_DATA_2: now also TP11.1
- net NES_LATCH: now also TP9.1
- net PWR_LED: now also R40.2; no longer U8.5 (LED_K)
- net RST_BTN: now also U8.4 (RST_OUT); no longer R40.2
- net VDAC_OUT: now also AV2.2; no longer AV2.1
- net at R40.1: now also U8.5 (LED_K); no longer U8.4 (RST_OUT)
- no-connect marks 17 -> 15
